File: imu-adaptor-board.sch (KiCad schematic (older format))
At the start: 3 parts, among them P1 IMU-CAN, P2 IMU-SPI3, U1 ADIS16405BMLZ

Commit message: add capacitor to power connector
Parts:
- added C1: 100n, imu-adaptor-board:0402, symbol C
Connections:
- net +5V: now also C1.1
- net GND: now also C1.2
Changed lines of the file:
@@
 Wire Wire Line
 	9600 3500 9500 3500
+$Comp
+L C C1
+U 1 1 56F17508
+P 1600 1600
+F 0 "C1" H 1625 1700 50  0000 L CNN
+F 1 "100n" H 1625 1500 50  0000 L CNN
+F 2 "imu-adaptor-board:0402" H 1638 1450 50  0001 C CNN
+F 3 "" H 1600 1600 50  0000 C CNN
+	1    1600 1600
+	1    0    0    -1
+$EndComp
+$Comp
+L +5V #PWR013
+U 1 1 56F175F5
+P 1600 1400
+F 0 "#PWR013" H 1600 1250 50  0001 C CNN
+F 1 "+5V" H 1600 1540 50  0000 C CNN
+F 2 "" H 1600 1400 50  0000 C CNN
+F 3 "" H 1600 1400 50  0000 C CNN
+	1    1600 1400
+	1    0    0    -1
+$EndComp
+$Comp
+L GND #PWR014
+U 1 1 56F1760C
+P 1600 1800
+F 0 "#PWR014" H 1600 1550 50  0001 C CNN
+F 1 "GND" H 1600 1650 50  0000 C CNN
+F 2 "" H 1600 1800 50  0000 C CNN
+F 3 "" H 1600 1800 50  0000 C CNN
+	1    1600 1800
+	1    0    0    -1
+$EndComp
+Wire Wire Line
+	1600 1800 1600 1750
+Wire Wire Line
+	1600 1450 1600 1400
 $EndSCHEMATC
